File: avionics  workshop.kicad_pcb (KiCad board)
At the start: 2 copper layers, 69.1 x 51 mm, 11 parts, among them U1 BMP280, U2 MPU-6050, U4 AMS1117-3.3

Commit message: draft1
Parts:
- D2: footprint LED_THT:LED_D5.0mm_Horizontal_O3.81mm_Z9.0mm -> LED_THT:LED_D5.0mm_Horizontal_O1.27mm_Z3.0mm
- moved D2 2.39 mm to (183.6, 67.3)
Routing:
- net Net-(D2-K): track 6.24 -> 8.67 mm
Changed lines of the file:
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@@
 	(net 55 "unconnected-(U2-RESV-Pad21)")
 	(net 56 "unconnected-(U2-AD0-Pad9)")
-	(footprint "LED_THT:LED_D5.0mm_Horizontal_O3.81mm_Z9.0mm"
+	(footprint "LED_THT:LED_D5.0mm_Horizontal_O1.27mm_Z3.0mm"
 		(layer "F.Cu")
-		(at 181.189 67.1626 90)
-		(descr "LED, diameter 5.0mm, horizontal offset 3.81mm, z-position of LED center 9.0mm, 2 pins, generated by kicad-footprint-generator")
+		(at 183.5766 67.2642 90)
+		(descr "LED, diameter 5.0mm, horizontal offset 1.27mm, z-position of LED center 3.0mm, 2 pins, generated by kicad-footprint-generator")
 		(tags "LED")
 		(property "Reference" "D2"
@@
 		)
 		(property "Value" "LED"
-			(at 1.27 13.47 90)
+			(at 1.27 10.93 90)
 			(layer "F.Fab")
 			(effects
@@
 		(fp_line
 			(start 2.54 1.08)
-			(end 2.54 3.75)
+			(end 2.54 1.21)
 			(stroke
 				(width 0.12)
@@
 		(fp_line
 			(start 0 1.08)
-			(end 0 3.75)
+			(end 0 1.21)
 			(stroke
 				(width 0.12)
@@
 		)
 		(fp_line
-			(start 4.23 3.75)
-			(end 4.23 4.87)
+			(start 4.23 1.21)
+			(end 4.23 2.33)
 			(stroke
 				(width 0.12)
@@
 		)
 		(fp_line
-			(start 3.83 3.75)
-			(end 4.23 3.75)
+			(start 3.83 1.21)
+			(end 4.23 1.21)
 			(stroke
 				(width 0.12)
@@
 		)
 		(fp_line
-			(start 3.83 3.75)
-			(end 3.83 9.91)
+			(start 3.83 1.21)
+			(end 3.83 7.37)
 			(stroke
 				(width 0.12)
@@
 		)
 		(fp_line
-			(start 2.54 3.75)
+			(start 2.54 1.21)
 			(end 2.54 1.08)
 			(stroke
@@
 		)
 		(fp_line
-			(start 2.54 3.75)
-			(end 2.54 3.75)
+			(start 2.54 1.21)
+			(end 2.54 1.21)
 			(stroke
 				(width 0.12)
@@
 		)
 		(fp_line
-			(start 0 3.75)
+			(start 0 1.21)
 			(end 0 1.08)
 			(stroke
@@
 		)
 		(fp_line
-			(start 0 3.75)
-			(end 0 3.75)
+			(start 0 1.21)
+			(end 0 1.21)
 			(stroke
 				(width 0.12)
@@
 		)
 		(fp_line
-			(start -1.29 3.75)
-			(end 3.83 3.75)
+			(start -1.29 1.21)
+			(end 3.83 1.21)
 			(stroke
 				(width 0.12)
@@
 		)
 		(fp_line
-			(start -1.29 3.75)
-			(end -1.29 9.91)
+			(start -1.29 1.21)
+			(end -1.29 7.37)
 			(stroke
 				(width 0.12)
@@
 		)
 		(fp_line
-			(start 4.23 4.87)
-			(end 3.83 4.87)
+			(start 4.23 2.33)
+			(end 3.83 2.33)
 			(stroke
 				(width 0.12)
@@
 		)
 		(fp_line
-			(start 3.83 4.87)
-			(end 3.83 3.75)
+			(start 3.83 2.33)
+			(end 3.83 1.21)
 			(stroke
 				(width 0.12)
@@
 		)
 		(fp_arc
-			(start 3.83 9.91)
-			(mid 1.27 12.47)
-			(end -1.29 9.91)
+			(start 3.83 7.37)
+			(mid 1.27 9.93)
+			(end -1.29 7.37)
 			(stroke
 				(width 0.12)
@@
 		(fp_line
 			(start -1.94 -1.21)
-			(end -1.94 12.72)
+			(end -1.94 10.18)
 			(stroke
 				(width 0.05)
@@
 		)
 		(fp_line
-			(start 4.49 12.72)
+			(start 4.49 10.18)
 			(end 4.49 -1.21)
 			(stroke
@@
 		)
 		(fp_line
-			(start -1.94 12.72)
-			(end 4.49 12.72)
+			(start -1.94 10.18)
+			(end 4.49 10.18)
 			(stroke
 				(width 0.05)
@@
 		(fp_line
 			(start 2.54 0)
-			(end 2.54 3.81)
+			(end 2.54 1.27)
 			(stroke
 				(width 0.1)
@@
 		(fp_line
 			(start 0 0)
-			(end 0 3.81)
+			(end 0 1.27)
 			(stroke
 				(width 0.1)
@@
 		)
 		(fp_line
-			(start 4.17 3.81)
-			(end 4.17 4.81)
+			(start 4.17 1.27)
+			(end 4.17 2.27)
 			(stroke
 				(width 0.1)
@@
 		)
 		(fp_line
-			(start 3.77 3.81)
-			(end 4.17 3.81)
+			(start 3.77 1.27)
+			(end 4.17 1.27)
 			(stroke
 				(width 0.1)
@@
 		)
 		(fp_line
-			(start 3.77 3.81)
-			(end 3.77 9.91)
+			(start 3.77 1.27)
+			(end 3.77 7.37)
 			(stroke
 				(width 0.1)
@@
 		)
 		(fp_line
-			(start 2.54 3.81)
+			(start 2.54 1.27)
 			(end 2.54 0)
 			(stroke
@@
 		)
 		(fp_line
-			(start 2.54 3.81)
-			(end 2.54 3.81)
+			(start 2.54 1.27)
+			(end 2.54 1.27)
 			(stroke
 				(width 0.1)
@@
 		)
 		(fp_line
-			(start 0 3.81)
+			(start 0 1.27)
 			(end 0 0)
 			(stroke
@@
 		)
 		(fp_line
-			(start 0 3.81)
-			(end 0 3.81)
+			(start 0 1.27)
+			(end 0 1.27)
 			(stroke
 				(width 0.1)
@@
 		)
 		(fp_line
-			(start -1.23 3.81)
-			(end 3.77 3.81)
+			(start -1.23 1.27)
+			(end 3.77 1.27)
 			(stroke
 				(width 0.1)
@@
 		)
 		(fp_line
-			(start -1.23 3.81)
-			(end -1.23 9.91)
+			(start -1.23 1.27)
+			(end -1.23 7.37)
 			(stroke
 				(width 0.1)
@@
 		)
 		(fp_line
-			(start 4.17 4.81)
-			(end 3.77 4.81)
+			(start 4.17 2.27)
+			(end 3.77 2.27)
 			(stroke
 				(width 0.1)
@@
 		)
 		(fp_line
-			(start 3.77 4.81)
-			(end 3.77 3.81)
+			(start 3.77 2.27)
+			(end 3.77 1.27)
 			(stroke
 				(width 0.1)
@@
 		)
 		(fp_arc
-			(start 3.77 9.91)
-			(mid 1.27 12.41)
-			(end -1.23 9.91)
+			(start 3.77 7.37)
+			(mid 1.27 9.87)
+			(end -1.23 7.37)
 			(stroke
 				(width 0.1)
@@
 		)
 		(fp_text user "${REFERENCE}"
-			(at 1.27 7.31 90)
+			(at 1.27 4.77 90)
 			(layer "F.Fab")
 			(effects
@@
 		)
 		(embedded_fonts no)
-		(model "${KICAD9_3DMODEL_DIR}/LED_THT.3dshapes/LED_D5.0mm_Horizontal_O3.81mm_Z9.0mm.step"
+		(model "${KICAD9_3DMODEL_DIR}/LED_THT.3dshapes/LED_D5.0mm_Horizontal_O1.27mm_Z3.0mm.step"
 			(offset
 				(xyz 0 0 0)
@@
 	(segment
 		(start 178.7158 64.6894)
-		(end 181.189 67.1626)
+		(end 181.2906 67.2642)
+		(width 0.8)
+		(layer "F.Cu")
+		(net 31)
+	)
+	(segment
+		(start 181.2906 67.2642)
+		(end 183.5766 67.2642)
 		(width 0.8)
 		(layer "F.Cu")

Commit message: draft2
Parts:
- removed U2: MPU-6050, Sensor_Motion:InvenSense_QFN-24_4x4mm_P0.5mm
- added G***: LOGO, sedsskillup:sedslogo, F.Cu at (187.9, 108.8)
- added MPU-6050: MPU-6050, GovindLibrary:MPU-6050, F.Cu at (158.7, 100.4)
- moved U1 9.70 mm to (151.8, 108.7), turned to 180 degrees
- moved R2 2.44 mm to (178.4, 66.7)
Connections:
- A1 pad 5: unconnected-(A1-D2-Pad5) -> /D2
Routing:
- net /D2: track 0.00 -> 45.5 mm
- net /SDA: track 21.3 -> 44.2 mm, vias 1 -> 2
- net /SCL: track 23.7 -> 43.3 mm, vias 3 -> 5
- net /SCK: track 41.4 -> 44.2 mm
- net /PWR(3.3): track 84.3 -> 86.9 mm, vias 5 -> 3
- net Net-(D2-K): track 8.67 -> 6.17 mm
- net /L2: track 55.5 -> 58.0 mm

Commit message: draft3
Routing:
- net /PWR(3.3): track 86.9 -> 90.6 mm
Changed lines of the file:
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@@
 	)
 	(segment
-		(start 150.0632 94.7236)
-		(end 154.552 99.2124)
+		(start 170.4848 96.7232)
+		(end 173.2788 96.7232)
+		(width 0.6)
+		(layer "F.Cu")
+		(net 34)
+	)
+	(segment
+		(start 170.3324 94.8944)
+		(end 170.4848 96.7232)
 		(width 0.6)
 		(layer "F.Cu")
@@
 	)
 	(segment
-		(start 154.552 99.2124)
-		(end 159.6822 99.2124)
+		(start 175.1076 94.9452)
+		(end 169.0116 88.8492)
 		(width 0.6)
 		(layer "F.Cu")
@@
 	)
 	(segment
-		(start 175.1076 94.9452)
-		(end 169.0116 88.8492)
+		(start 150.0632 94.7236)
+		(end 150.0632 99.2124)
 		(width 0.6)
 		(layer "F.Cu")
@@
 	)
 	(segment
-		(start 168.148 87.9856)
-		(end 168.148 87.122)
+		(start 150.0632 99.2124)
+		(end 159.6822 99.2124)
 		(width 0.6)
 		(layer "F.Cu")
@@
 	)
 	(segment
-		(start 171.8846 96.4466)
-		(end 173.6066 96.4466)
+		(start 173.2788 96.7232)
+		(end 175.1076 94.9456)
+		(width 0.6)
+		(layer "F.Cu")
+		(net 34)
+	)
+	(segment
+		(start 168.148 87.9856)
+		(end 168.148 87.122)
 		(width 0.6)
 		(layer "F.Cu")
@@
 		(start 175.1076 85.2932)
 		(end 175.1076 88.6456)
-		(width 0.6)
-		(layer "F.Cu")
-		(net 34)
-	)
-	(segment
-		(start 170.3324 94.8944)
-		(end 171.8846 96.4466)
-		(width 0.6)
-		(layer "F.Cu")
-		(net 34)
-	)
-	(segment
-		(start 173.6066 96.4466)
-		(end 175.1076 94.9456)
 		(width 0.6)
 		(layer "F.Cu")
@@
 	)
 	(segment
-		(start 163.734011 85.852)
-		(end 161.798 85.852)
+		(start 170.0784 92.2528)
+		(end 170.0784 92.196389)
+		(width 0.6)
+		(layer "B.Cu")
+		(net 34)
+	)
+	(segment
+		(start 170.3324 94.8944)
+		(end 170.0784 92.2528)
+		(width 0.6)
+		(layer "B.Cu")
+		(net 34)
+	)
+	(segment
+		(start 169.9768 85.2932)
+		(end 175.1076 85.2932)
 		(width 0.6)
 		(layer "B.Cu")
@@
 		(start 170.0784 92.196389)
 		(end 163.734011 85.852)
-		(width 0.6)
-		(layer "B.Cu")
-		(net 34)
-	)
-	(segment
-		(start 170.3324 94.8944)
-		(end 170.18 92.202)
-		(width 0.6)
-		(layer "B.Cu")
-		(net 34)
-	)
-	(segment
-		(start 169.9768 85.2932)
-		(end 175.1076 85.2932)
 		(width 0.6)
 		(layer "B.Cu")
@@
 	)
 	(segment
-		(start 170.18 92.202)
-		(end 170.0784 92.196389)
+		(start 163.734011 85.852)
+		(end 161.798 85.852)
 		(width 0.6)
 		(layer "B.Cu")

Commit message: draft4
Parts:
- removed MPU-6050: MPU-6050, GovindLibrary:MPU-6050
- added U2: ~, GovindLibrary:MPU-6050, F.Cu at (158.6, 100.3)
- added U5: ~, GovindLibrary:AS32-TTL100, F.Cu at (175.5, 116.4)
- moved G*** 18.0 mm to (192.8, 91.5)
Connections:
- A1 pad 1: unconnected-(A1-D1/TX-Pad1) -> /RXD
- A1 pad 2: unconnected-(A1-D0/RX-Pad2) -> /TXD
Routing:
- net /TXD: track 0.00 -> 77.9 mm
- net /RXD: track 0.00 -> 62.2 mm, vias 0 -> 3
- net +5V: track 63.7 -> 86.8 mm
- net /PWR(3.3): track 90.6 -> 92.7 mm
- net /SCL: track 43.3 -> 43.9 mm
Other:
- board size 69.1 x 51 mm -> 69.7 x 64.8 mm

Commit message: draft7
Parts:
- U1: footprint Package_LGA:Bosch_LGA-8_2x2.5mm_P0.65mm_ClockwisePinNumbering -> GovindLibrary:BMP280
- U4: footprint Package_TO_SOT_SMD:SOT-223-3_TabPin2 -> GovindLibrary:AMS-1117
- moved U1 12.7 mm to (141.1, 115.5)
- moved U4 6.20 mm to (181.1, 93.4)
Connections:
- U1 pad 1: GND -> /PWR(3.3)
- U1 pad 3: /SDA -> /SCL
- U1 pad 4: /SCL -> /SDA
- U4 pad 1: GND -> +5V
- U4 pad 3: +5V -> GND
Routing:
- net /D2: track 45.0 -> 76.9 mm, vias 0 -> 1
- net /SCL: track 43.9 -> 62.6 mm
- net /SDA: track 44.5 -> 57.8 mm
- net /PWR(3.3): track 92.7 -> 81.5 mm, vias 3 -> 2
- net +5V: track 86.8 -> 97.3 mm
- net /L2: track 58.0 -> 65.1 mm
- net /cs: track 46.9 -> 49.3 mm
- net /SCK: track 44.2 -> 46.7 mm
- net /L3: track 56.0 -> 58.0 mm
- net /TXD: track 77.9 -> 79.5 mm, vias 0 -> 2
- net /MISO: track 40.2 -> 41.1 mm
