File: avionics  workshop.kicad_sch (KiCad schematic)
At the start: 11 parts, among them U1 BMP280, U2 MPU-6050, U4 AMS1117-3.3

Commit message: draft1
Parts:
- D2: footprint LED_THT:LED_D5.0mm_Horizontal_O3.81mm_Z9.0mm -> LED_THT:LED_D5.0mm_Horizontal_O1.27mm_Z3.0mm
Changed lines of the file:
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@@
 			)
 		)
-		(property "Footprint" "LED_THT:LED_D5.0mm_Horizontal_O3.81mm_Z9.0mm"
+		(property "Footprint" "LED_THT:LED_D5.0mm_Horizontal_O1.27mm_Z3.0mm"
 			(at 44.45 83.82 0)
 			(effects

Commit message: draft2
Parts:
- removed U2: MPU-6050, Sensor_Motion:InvenSense_QFN-24_4x4mm_P0.5mm, symbol Sensor_Motion:MPU-6050
- added U2: ~, symbol New_Library:MPU-6050
Connections:
- net GND: now also U2.2 (Gnd), U2.7 (ADO)
- net PWR(3.3): now also U2. (Vcc)
- net SCL: now also U2.3 (SCL)
- net SDA: now also U2.4 (SDA)
- net D2: now reaches A1.5 (D2)
- net D2: now also U2.8 (INT)
- no-connect marks 31 -> 22
Changed lines of the file:
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@@
-	)
-	(no_connect
-		(at 209.55 63.5)
 	)
 	(no_connect
@@
 	)
 	(no_connect
-		(at 229.87 88.9)
-	)
-	(no_connect
 		(at 96.52 83.82)
 	)
@@
 	)
 	(no_connect
-		(at 194.31 86.36)
-	)
-	(no_connect
 		(at 165.1 82.55)
 	)
@@
 	)
 	(no_connect
-		(at 229.87 86.36)
-	)
-	(no_connect
-		(at 229.87 81.28)
-	)
-	(no_connect
 		(at 139.7 90.17)
 	)
@@
 	)
 	(no_connect
-		(at 194.31 78.74)
-	)
-	(no_connect
-		(at 229.87 73.66)
+		(at 203.2 81.28)
 	)
 	(no_connect
@@
 	)
 	(no_connect
-		(at 139.7 72.39)
-	)
-	(no_connect
-		(at 194.31 88.9)
-	)
-	(no_connect
 		(at 139.7 67.31)
 	)
 	(no_connect
-		(at 229.87 78.74)
-	)
-	(no_connect
 		(at 165.1 90.17)
 	)
@@
 	(wire
 		(pts
+			(xy 196.85 83.82) (xy 196.85 95.25)
+		)
+		(stroke
+			(width 0)
+			(type default)
+		)
+	)
+	(wire
+		(pts
 			(xy 165.1 92.71) (xy 176.53 92.71)
 		)
@@
 	(wire
 		(pts
+			(xy 134.62 72.39) (xy 139.7 72.39)
+		)
+		(stroke
+			(width 0)
+			(type default)
+		)
+	)
+	(wire
+		(pts
 			(xy 191.77 77.47) (xy 194.31 77.47)
 		)
@@
 	(wire
 		(pts
-			(xy 191.77 73.66) (xy 194.31 73.66)
+			(xy 200.66 78.74) (xy 203.2 78.74)
 		)
 		(stroke
@@
 	(wire
 		(pts
+			(xy 203.2 83.82) (xy 196.85 83.82)
+		)
+		(stroke
+			(width 0)
+			(type default)
+		)
+	)
+	(wire
+		(pts
 			(xy 265.43 88.9) (xy 262.89 88.9)
 		)
@@
 	(wire
 		(pts
+			(xy 196.85 95.25) (xy 212.09 95.25)
+		)
+		(stroke
+			(width 0)
+			(type default)
+		)
+	)
+	(wire
+		(pts
 			(xy 151.13 111.76) (xy 151.13 114.3)
 		)
@@
 	(wire
 		(pts
+			(xy 194.31 76.2) (xy 203.2 76.2)
+		)
+		(stroke
+			(width 0)
+			(type default)
+		)
+	)
+	(wire
+		(pts
 			(xy 151.13 111.76) (xy 152.4 111.76)
 		)
@@
 	(wire
 		(pts
-			(xy 214.63 58.42) (xy 214.63 63.5)
-		)
-		(stroke
-			(width 0)
-			(type default)
-		)
-	)
-	(wire
-		(pts
 			(xy 67.31 68.58) (xy 72.39 68.58)
 		)
@@
 	(wire
 		(pts
+			(xy 200.66 86.36) (xy 203.2 86.36)
+		)
+		(stroke
+			(width 0)
+			(type default)
+		)
+	)
+	(wire
+		(pts
 			(xy 36.83 73.66) (xy 39.37 73.66)
 		)
@@
 	(wire
 		(pts
+			(xy 212.09 90.17) (xy 212.09 95.25)
+		)
+		(stroke
+			(width 0)
+			(type default)
+		)
+	)
+	(wire
+		(pts
 			(xy 250.19 91.44) (xy 250.19 92.71)
 		)
@@
 	(wire
 		(pts
+			(xy 212.09 67.31) (xy 212.09 71.12)
+		)
+		(stroke
+			(width 0)
+			(type default)
+		)
+	)
+	(wire
+		(pts
 			(xy 250.19 72.39) (xy 262.89 72.39)
 		)
@@
 		(pts
 			(xy 109.22 91.44) (xy 109.22 93.98)
-		)
-		(stroke
-			(width 0)
-			(type default)
-		)
-	)
-	(wire
-		(pts
-			(xy 215.9 58.42) (xy 214.63 58.42)
 		)
 		(stroke
@@
 		)
 	)
+	(label "PWR(3.3)"
+		(at 212.09 67.31 0)
+		(effects
+			(font
+				(size 1.27 1.27)
+			)
+			(justify left bottom)
+		)
+	)
 	(label "GND"
 		(at 107.95 93.98 270)
@@
 		)
 	)
+	(label "D2"
+		(at 200.66 86.36 0)
+		(effects
+			(font
+				(size 1.27 1.27)
+			)
+			(justify left bottom)
+		)
+	)
 	(label "L2"
 		(at 130.81 85.09 0)
@@
 	)
 	(label "PWR(3.3)"
-		(at 215.9 58.42 0)
-		(effects
-			(font
-				(size 1.27 1.27)
-			)
-			(justify left bottom)
-		)
-	)
-	(label "PWR(3.3)"
 		(at 274.32 81.28 270)
 		(effects
@@
 	)
 	(label "GND"
-		(at 212.09 99.06 270)
+		(at 212.09 95.25 270)
 		(effects
 			(font
@@
 	)
 	(label "SDA"
-		(at 191.77 73.66 180)
+		(at 200.66 78.74 180)
 		(effects
 			(font
@@
 		)
 	)
+	(label "D2"
+		(at 134.62 72.39 0)
+		(effects
+			(font
+				(size 1.27 1.27)
+			)
+			(justify left bottom)
+		)
+	)
 	(label "GND"
 		(at 265.43 88.9 0)
@@
 			)
 			(justify left bottom)
-		)
-	)
-	(symbol
-		(lib_id "Sensor_Motion:MPU-6050")
-		(at 212.09 81.28 0)
-		(unit 1)
-		(exclude_from_sim no)
-		(in_bom yes)
-		(on_board yes)
-		(dnp no)
-		(fields_autoplaced yes)
-		(property "Reference" "U2"
-			(at 214.2333 97.79 0)
-			(effects
-				(font
-					(size 1.27 1.27)
-				)
-				(justify left)
-			)
-		)
-		(property "Value" "MPU-6050"
-			(at 214.2333 100.33 0)
-			(effects
-				(font
-					(size 1.27 1.27)
-				)
-				(justify left)
-			)
-		)
-		(property "Footprint" "Sensor_Motion:InvenSense_QFN-24_4x4mm_P0.5mm"
-			(at 212.09 101.6 0)
-			(effects
-				(font
-					(size 1.27 1.27)
-				)
-				(hide yes)
-			)
-		)
-		(property "Datasheet" "https://invensense.tdk.com/wp-content/uploads/2015/02/MPU-6000-Datasheet1.pdf"
-			(at 212.09 85.09 0)
-			(effects
-				(font
-					(size 1.27 1.27)
-				)
-				(hide yes)
-			)
-		)
-		(property "Description" "InvenSense 6-Axis Motion Sensor, Gyroscope, Accelerometer, I2C"
-			(at 212.09 81.28 0)
-			(effects
-				(font
-					(size 1.27 1.27)
-				)
-				(hide yes)
-			)
-		)
-		(pin "18"
-		)
-		(pin "3"
-		)
-		(pin "14"
-		)
-		(pin "16"
-		)
-		(pin "11"
-		)
-		(pin "4"
-		)
-		(pin "13"
-		)
-		(pin "1"
-		)
-		(pin "21"
-		)
-		(pin "22"
-		)
-		(pin "17"
-		)
-		(pin "2"
-		)
-		(pin "9"
-		)
-		(pin "8"
-		)
-		(pin "5"
-		)
-		(pin "23"
-		)
-		(pin "15"
-		)
-		(pin "24"
-		)
-		(pin "19"
-		)
-		(pin "7"
-		)
-		(pin "20"
-		)
-		(pin "12"
-		)
-		(pin "10"
-		)
-		(pin "6"
-		)
-		(instances
-			(project ""
-				(path "/b922d51f-b961-4ded-8569-767b32b1ff85"
-					(reference "U2")
-					(unit 1)
-				)
-			)
 		)
 	)
@@
 					(unit 1)
 				)
+			)
+		)
+	)
+	(symbol
+		(lib_id "New_Library:MPU-6050")
+		(at 210.82 81.28 0)
+		(unit 1)
+		(exclude_from_sim no)
+		(in_bom yes)
+		(on_board yes)
+		(dnp no)
+		(fields_autoplaced yes)
+		(property "Reference" "U2"
+			(at 218.44 80.0099 0)
+			(effects
+				(font
+					(size 1.27 1.27)
+				)
+				(justify left)
+			)
+		)
+		(property "Value" "~"
+			(at 218.44 81.915 0)
+			(effects
+				(font
+					(size 1.27 1.27)
+				)
+				(justify left)
+			)
+		)
+		(property "Footprint" ""
+			(at 210.82 81.28 0)
+			(effects
+				(font
+					(size 1.27 1.27)
+				)
+				(hide yes)
+			)
+		)
+		(property "Datasheet" ""
+			(at 210.82 81.28 0)
+			(effects
+				(font
+					(size 1.27 1.27)
+				)
+				(hide yes)
+			)
+		)
+		(property "Description" ""
+			(at 210.82 81.28 0)
+			(effects
+				(font
+					(size 1.27 1.27)
+				)
+				(hide yes)
+			)
+		)
+		(pin "6"
+		)
+		(pin "4"
+		)
+		(pin "3"
+		)
+		(pin "7"
+		)
+		(pin "8"
+		)
+		(pin ""
+		)
+		(pin "2"
+		)
+		(instances
+			(project ""
+				(path "/b922d51f-b961-4ded-8569-767b32b1ff85"
+					(reference "U2")
+					(unit 1)
+				)

Commit message: draft4
Parts:
- added U5: ~, GovindLibrary:AS32-TTL100, symbol New_Library:AS32-TTL100
- U2: footprint (none) -> GovindLibrary:MPU-6050
Connections:
- net +5V: now also U5.6 (Vcc)
- net GND: now also U5.1 (MD0), U5.2 (MD1), U5.7 (Gnd)
- net RXD: now reaches A1.1 (D1/TX)
- net RXD: now also U5.3 (RXD)
- net TXD: now reaches A1.2 (D0/RX)
- net TXD: now also U5.4 (TXD)
- no-connect marks 22 -> 21
Other:
- note added: "AS32-ttl 100"

Commit message: draft7
Parts:
- removed U4: AMS1117-3.3, Package_TO_SOT_SMD:SOT-223-3_TabPin2, symbol Regulator_Linear:AMS1117-3.3
- added U4: AMS1117CD-3.3, GovindLibrary:AMS-1117, symbol Regulator_Linear:AMS1117CD-3.3
- U1: footprint Package_LGA:Bosch_LGA-8_2x2.5mm_P0.65mm_ClockwisePinNumbering -> GovindLibrary:BMP280
Connections:
- net +5V: now also U4.3 (VI)
- net GND: now also U4.1 (GND)
- net PWR(3.3): now also U4.2 (VO)
Other:
- moved on the sheet: U5
Changed lines of the file:
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@@
 	)
 	(rectangle
-		(start 35.56 133.096)
-		(end 70.866 181.102)
+		(start 243.84 112.776)
+		(end 279.146 160.782)
 		(stroke
 			(width 0)
@@
 	(text "AS32-ttl 100"
 		(exclude_from_sim no)
-		(at 53.34 129.794 0)
+		(at 262.382 111.252 0)
 		(effects
 			(font
@@
 	)
 	(no_connect
-		(at 58.42 146.05)
+		(at 266.7 125.73)
 	)
 	(no_connect
@@
 	(wire
 		(pts
-			(xy 55.88 138.43) (xy 55.88 146.05)
+			(xy 264.16 118.11) (xy 264.16 125.73)
 		)
 		(stroke
@@
 	(wire
 		(pts
-			(xy 53.34 135.89) (xy 53.34 146.05)
+			(xy 261.62 115.57) (xy 261.62 125.73)
 		)
 		(stroke
@@
 	(wire
 		(pts
-			(xy 48.26 140.97) (xy 48.26 146.05)
+			(xy 256.54 120.65) (xy 256.54 125.73)
 		)
 		(stroke
@@
 	(wire
 		(pts
-			(xy 57.15 162.56) (xy 57.15 167.64)
+			(xy 265.43 142.24) (xy 265.43 147.32)
 		)
 		(stroke
@@
 	(wire
 		(pts
-			(xy 49.53 162.56) (xy 49.53 167.64)
+			(xy 257.81 142.24) (xy 257.81 147.32)
 		)
 		(stroke
@@
 	(wire
 		(pts
-			(xy 50.8 143.51) (xy 50.8 146.05)
+			(xy 259.08 123.19) (xy 259.08 125.73)
 		)
 		(stroke
@@
 	)
 	(label "RXD"
-		(at 53.34 135.89 0)
+		(at 261.62 115.57 0)
 		(effects
 			(font
@@
 	)
 	(label "GND"
-		(at 49.53 167.64 270)
+		(at 257.81 147.32 270)
 		(effects
 			(font
@@
 	)
 	(label "GND"
-		(at 48.26 140.97 0)
+		(at 256.54 120.65 0)
 		(effects
 			(font
@@
 	)
 	(label "GND"
-		(at 50.8 143.51 0)
+		(at 259.08 123.19 0)
 		(effects
 			(font
@@
 	)
 	(label "TXD"
-		(at 55.88 138.43 0)
+		(at 264.16 118.11 0)
 		(effects
 			(font
@@
 	(symbol
 		(lib_id "New_Library:AS32-TTL100")
-		(at 53.34 153.67 0)
+		(at 261.62 133.35 0)
 		(unit 1)
 		(exclude_from_sim no)
@@
 		(fields_autoplaced yes)
 		(property "Reference" "U5"
-			(at 60.96 153.6699 0)
+			(at 269.24 133.3499 0)
 			(effects
 				(font
@@
 		)
 		(property "Value" "~"
-			(at 60.96 155.575 0)
+			(at 269.24 135.255 0)
 			(effects
 				(font
@@
 		)
 		(property "Footprint" "GovindLibrary:AS32-TTL100"
-			(at 53.34 153.67 0)
+			(at 261.62 133.35 0)
 			(effects
 				(font
@@
 		)
 		(property "Datasheet" ""
-			(at 53.34 153.67 0)
+			(at 261.62 133.35 0)
 			(effects
 				(font
@@
 		)
 		(property "Description" ""
-			(at 53.34 153.67 0)
+			(at 261.62 133.35 0)
 			(effects
 				(font
@@
 	(symbol
 		(lib_id "power:+5V")
-		(at 57.15 167.64 180)
+		(at 265.43 147.32 180)
 		(unit 1)
 		(exclude_from_sim no)
@@
 		(fields_autoplaced yes)
 		(property "Reference" "#PWR06"
-			(at 57.15 163.83 0)
+			(at 265.43 143.51 0)
 			(effects
 				(font
@@
 		)
 		(property "Value" "+5V"
-			(at 57.15 172.72 0)
+			(at 265.43 152.4 0)
 			(effects
 				(font
@@
 		)
 		(property "Footprint" ""
-			(at 57.15 167.64 0)
+			(at 265.43 147.32 0)
 			(effects
 				(font
@@
 		)
 		(property "Datasheet" ""
-			(at 57.15 167.64 0)
+			(at 265.43 147.32 0)
 			(effects
 				(font
@@
 		)
 		(property "Description" "Power symbol creates a global label with name \"+5V\""
-			(at 57.15 167.64 0)
+			(at 265.43 147.32 0)
 			(effects
 				(font
@@
 				(path "/b922d51f-b961-4ded-8569-767b32b1ff85"
 					(reference "A1")
-					(unit 1)
-				)
-			)
-		)
-	)
-	(symbol
-		(lib_id "Regulator_Linear:AMS1117-3.3")
-		(at 262.89 81.28 0)
-		(unit 1)
-		(exclude_from_sim no)
-		(in_bom yes)
-		(on_board yes)
-		(dnp no)
-		(fields_autoplaced yes)
-		(property "Reference" "U4"
-			(at 262.89 74.93 0)
-			(effects
-				(font
-					(size 1.27 1.27)
-				)
-			)
-		)
-		(property "Value" "AMS1117-3.3"
-			(at 262.89 77.47 0)
-			(effects
-				(font
-					(size 1.27 1.27)
-				)
-			)
-		)
-		(property "Footprint" "Package_TO_SOT_SMD:SOT-223-3_TabPin2"
-			(at 262.89 76.2 0)
-			(effects
-				(font
-					(size 1.27 1.27)
-				)
-				(hide yes)
-			)
-		)
-		(property "Datasheet" "http://www.advanced-monolithic.com/pdf/ds1117.pdf"
-			(at 265.43 87.63 0)
-			(effects
-				(font
-					(size 1.27 1.27)
-				)
-				(hide yes)
-			)
-		)
-		(property "Description" "1A Low Dropout regulator, positive, 3.3V fixed output, SOT-223"
-			(at 262.89 81.28 0)
-			(effects
-				(font
-					(size 1.27 1.27)
-				)
-				(hide yes)
-			)
-		)
-		(pin "3"
-		)
-		(pin "1"
-		)
-		(pin "2"
-		)
-		(instances
-			(project ""
-				(path "/b922d51f-b961-4ded-8569-767b32b1ff85"
-					(reference "U4")
 					(unit 1)
 				)
@@
 	)
 	(symbol
+		(lib_id "Regulator_Linear:AMS1117CD-3.3")
+		(at 262.89 81.28 0)
+		(unit 1)
+		(exclude_from_sim no)
+		(in_bom yes)
+		(on_board yes)
+		(dnp no)
+		(fields_autoplaced yes)
+		(property "Reference" "U4"
+			(at 262.89 74.93 0)
+			(effects
+				(font
+					(size 1.27 1.27)
+				)
+			)
+		)
+		(property "Value" "AMS1117CD-3.3"
+			(at 262.89 77.47 0)
+			(effects
+				(font
+					(size 1.27 1.27)
+				)
+			)
+		)
+		(property "Footprint" "GovindLibrary:AMS-1117"
+			(at 262.89 76.2 0)
+			(effects
+				(font
+					(size 1.27 1.27)
+				)
+				(hide yes)
+			)
+		)
+		(property "Datasheet" "http://www.advanced-monolithic.com/pdf/ds1117.pdf"
+			(at 265.43 87.63 0)
+			(effects
+				(font
+					(size 1.27 1.27)
+				)
+				(hide yes)
+			)
+		)
+		(property "Description" "1A Low Dropout regulator, positive, 3.3V fixed output, TO-252"
+			(at 262.89 81.28 0)
+			(effects
+				(font
+					(size 1.27 1.27)
+				)
+				(hide yes)
+			)
+		)
+		(pin "2"
+		)
+		(pin "1"
+		)
+		(pin "3"
+		)
+		(instances
+			(project ""
+				(path "/b922d51f-b961-4ded-8569-767b32b1ff85"
+					(reference "U4")
+					(unit 1)
+				)
+			)
+		)
+	)
+	(symbol
 		(lib_id "power:PWR_FLAG")
 		(at 52.07 97.79 90)
@@
 			)
 		)
-		(property "Footprint" "Package_LGA:Bosch_LGA-8_2x2.5mm_P0.65mm_ClockwisePinNumbering"
+		(property "Footprint" "GovindLibrary:BMP280"
 			(at 106.68 101.6 0)
 			(effects
